Commit message: adding docking

File: yuki_robot_description/urdf/robot.urdf (robot description, URDF)
Before this commit: robot yuki_bot, 6 links, 9 joints
Links:
- removed link camera_depth_frame
- added link cam_1_depth_frame
- added link cam_1_depth_optical_frame
Joints:
- added joint cam_1_depth_optical_joint: type fixed, parent cam_1_depth_frame, child cam_1_depth_optical_frame, origin xyz=0 0 0 rpy=${-pi/2} 0 ${-pi/2}
- joint camera_depth_joint: child camera_depth_frame -> cam_1_depth_frame
